Commit message: Update lidar link name and orientation, changed lidar frame name to laser to support OM1

File: go2_gazebo_sim/go2_description/urdf/velodyne.xacro (robot description, xacro)
@@ -32,7 +32,7 @@
         <origin rpy="0 0 0" xyz="0 0 0.0377"/>
         <parent link="velodyne_base_link"/>
-        <child link="velodyne"/>
+        <child link="laser"/>
     </joint>
-    <link name="velodyne">
+    <link name="laser">
         <inertial>
             <mass value="0.01"/>
@@ -48,9 +48,10 @@
     </link>
     <!-- Gazebo Sim Velodyne Sensor plugin -->
-    <gazebo reference="velodyne">
+    <gazebo reference="laser">
         <sensor name="velodyne-VLP16" type="gpu_lidar">
+            <pose>0 0 0 0 0 3.14159</pose>
             <topic>scan</topic>
             <update_rate>10</update_rate>
-            <gz_frame_id>velodyne</gz_frame_id>
+            <gz_frame_id>laser</gz_frame_id>
             <lidar>
                 <scan>
@@ -78,5 +79,5 @@
                     <stddev>0.008</stddev>
                 </noise>
-                <frame_id>velodyne</frame_id>
+                <frame_id>laser</frame_id>
             </lidar>
             <visualize>true</visualize>
