Commit message: Add simulated RealSense D435 camera to Go2 robot with Gazebo sensors and ROS bridge topics.

File: go2_gazebo_sim/go2_description/urdf/unitree_go2_gazebo.xacro (robot description, xacro)
@@ -117,4 +117,46 @@
     </sensor>
   </gazebo>
+  <!-- Head Camera Plugin (Downfacing RealSense) -->
+  <gazebo reference="camera_link">
+    <sensor name="head_depth_camera" type="depth_camera">
+      <pose>0 0 0 0 0 0</pose>
+      <camera>
+        <horizontal_fov>1.518</horizontal_fov> <!-- RealSense D435i approx FOV -->
+        <image>
+          <width>640</width>
+          <height>480</height>
+        </image>
+        <clip>
+          <near>0.1</near>
+          <far>10.0</far>
+        </clip>
+      </camera>
+      <gz_frame_id>camera_link</gz_frame_id>
+      <always_on>1</always_on>
+      <update_rate>30</update_rate>
+      <visualize>1</visualize>
+      <topic>camera/realsense2_camera_node/depth/image_rect_raw</topic>
+    </sensor>
+    <sensor name="head_rgb_camera" type="camera">
+      <pose>0 0 0 0 0 0</pose>
+      <camera>
+        <horizontal_fov>1.518</horizontal_fov>
+        <image>
+          <width>640</width>
+          <height>480</height>
+          <format>R8G8B8</format>
+        </image>
+        <clip>
+          <near>0.05</near>
+          <far>10.0</far>
+        </clip>
+      </camera>
+      <gz_frame_id>camera_link</gz_frame_id>
+      <always_on>1</always_on>
+      <update_rate>30</update_rate>
+      <visualize>1</visualize>
+      <topic>camera/realsense2_camera_node/color/image_raw</topic>
+    </sensor>
+  </gazebo>
   <!-- Main body -->
   <gazebo reference="trunk">

File: go2_gazebo_sim/go2_description/urdf/unitree_go2_robot.xacro (robot description, xacro)
@@ -79,24 +79,21 @@
         </collision>
     </link>
-    <!-- Camera Link-->
+    <!-- Camera Link (Downfacing RealSense) -->
     <link name="camera_link">
         <inertial>
-            <mass value="0.001"/>
+            <mass value="0.01"/>
             <origin rpy="0 0 0" xyz="0 0 0"/>
             <inertia ixx="0.0001" ixy="0" ixz="0" iyy="0.0001" iyz="0" izz="0.0001"/>
         </inertial>
         <visual>
-            <origin rpy="0 0 0" xyz="0 0 0"/>
+            <origin rpy="1.57 0 1.57" xyz="0.01 0 0"/>
             <geometry>
-                <sphere radius="0.001"/>
+                <mesh filename="file://$(find go2_description)/meshes/d435.dae" scale="1 1 1"/>
             </geometry>
-            <material name="">
-                <color rgba="0.5 0 0 1" />
-            </material>
         </visual>
         <collision>
             <origin rpy="0 0 0" xyz="0 0 0"/>
             <geometry>
-                <sphere radius="0.001"/>
+                <box size="0.025 0.09 0.025"/>
             </geometry>
         </collision>
@@ -105,5 +102,5 @@
         <parent link="trunk"/>
         <child link="camera_link"/>
-        <origin rpy="0 0 0" xyz="0.326 0 0.043"/>
+        <origin rpy="0 0.5236 0" xyz="0.326 0 0.043"/>
     </joint>
     <!-- <joint name="lidar_l1_joint" type="fixed">

Commit message: Fix multiple issues

File: go2_gazebo_sim/go2_description/urdf/unitree_go2_gazebo.xacro (robot description, xacro)
@@ -120,21 +120,49 @@
   <gazebo reference="camera_link">
     <sensor name="head_depth_camera" type="depth_camera">
-      <pose>0 0 0 0 0 0</pose>
+      <pose>0.02 0 0 0 0 0</pose>
       <camera>
-        <horizontal_fov>1.518</horizontal_fov> <!-- RealSense D435i approx FOV -->
+        <lens>
+          <intrinsics>
+            <fx>242.479</fx>
+            <fy>242.479</fy>
+            <cx>242.736</cx>
+            <cy>133.273</cy>
+            <s>0</s>
+          </intrinsics>
+        </lens>
+        <distortion>
+          <k1>0.0</k1>
+          <k2>0.0</k2>
+          <k3>0.0</k3>
+          <p1>0.0</p1>
+          <p2>0.0</p2>
+          <center>0.5 0.5</center>
+        </distortion>
         <image>
-          <width>640</width>
-          <height>480</height>
+          <width>480</width>
+          <height>270</height>
+          <format>R8G8B8</format>
         </image>
         <clip>
-          <near>0.1</near>
-          <far>10.0</far>
+          <near>0.01</near>
+          <far>300</far>
         </clip>
+        <depth_camera>
+          <clip>
+            <near>0.1</near>
+            <far>10</far>
+          </clip>
+        </depth_camera>
+        <noise>
+          <type>gaussian</type>
+          <mean>0</mean>
+          <stddev>0.003</stddev>
+        </noise>
       </camera>
       <gz_frame_id>camera_link</gz_frame_id>
       <always_on>1</always_on>
-      <update_rate>30</update_rate>
+      <update_rate>10</update_rate>
       <visualize>1</visualize>
-      <topic>camera/realsense2_camera_node/depth/image_rect_raw</topic>
+      <topic>camera/realsense2_camera_node/depth/image_rect_gazebo_raw</topic>
     </sensor>
     <sensor name="head_rgb_camera" type="camera">

File: go2_gazebo_sim/go2_description/urdf/unitree_go2_robot.xacro (robot description, xacro)
@@ -102,5 +102,5 @@
         <parent link="trunk"/>
         <child link="camera_link"/>
-        <origin rpy="0 0.5236 0" xyz="0.326 0 0.043"/>
+        <origin rpy="0 0.6109 0" xyz="0.33 0 0.065"/>
     </joint>
     <!-- <joint name="lidar_l1_joint" type="fixed">
