Commit message: Support OM1

File: go2_gazebo_sim/go2_description/urdf/unitree_go2_robot.xacro (robot description, xacro)
@@ -102,5 +102,5 @@
         <parent link="trunk"/>
         <child link="camera_link"/>
-        <origin rpy="0 0.6109 0" xyz="0.33 0 0.065"/>
+        <origin rpy="0 0.6109 0" xyz="0.33 0 0.085"/>
     </joint>
     <!-- <joint name="lidar_l1_joint" type="fixed">
