Commit message: Enable multi-robot simulation with namespacing, joystick control, and new launch/RVIZ configurations.

File: go2_gazebo_sim/go2_description/urdf/lidar_4D_lidar.xacro (robot description, xacro)
@@ -35,5 +35,5 @@
     <gazebo reference="lidar_l1_link">
         <sensor name="lidar_l1" type="gpu_lidar">
-            <topic>unitree_lidar</topic>
+            <topic>${topic_prefix}unitree_lidar</topic>
             <update_rate>10</update_rate>
             <lidar>

File: go2_gazebo_sim/go2_description/urdf/unitree_go2_gazebo.xacro (robot description, xacro)
@@ -1,4 +1,4 @@
 <?xml version="1.0"?>
-<robot>
+<robot xmlns:xacro="http://www.ros.org/wiki/xacro">
   <!-- Gazebo Sim plugins -->
   <gazebo>
@@ -26,5 +26,11 @@
     <plugin filename="gz_ros2_control-system" name="gz_ros2_control::GazeboSimROS2ControlPlugin">
       <parameters>$(find go2_gazebo_sim)/config/ros_control/ros_control.yaml</parameters>
+      <!-- When namespace is set, the plugin runs in that namespace, so robot_param_node should be relative -->
       <robot_param_node>robot_state_publisher</robot_param_node>
+      <xacro:if value="${ns != ''}">
+        <ros>
+          <namespace>${ns}</namespace>
+        </ros>
+      </xacro:if>
     </plugin>
   </gazebo>
@@ -33,9 +39,9 @@
   <plugin filename="libignition-gazebo-odometry-publisher-system.so"
           name="ignition::gazebo::systems::OdometryPublisher">
-      <odom_frame>odom</odom_frame>
-      <robot_base_frame>base_link</robot_base_frame>
-      <odom_topic>/odom</odom_topic>
+      <odom_frame>${topic_prefix}odom</odom_frame>
+      <robot_base_frame>${topic_prefix}base_link</robot_base_frame>
+      <odom_topic>${topic_prefix}odom</odom_topic>
       <odom_publish_frequency>50</odom_publish_frequency>
-      <tf_topic>/tf</tf_topic>
+      <tf_topic>${topic_prefix}tf</tf_topic>
     </plugin>
   </gazebo>
@@ -46,5 +52,5 @@
       <update_rate>100</update_rate>
       <visualize>true</visualize>
-      <topic>imu/data</topic>
+      <topic>${topic_prefix}imu/data</topic>
       <gz_frame_id>imu_link</gz_frame_id>
       <imu>
@@ -114,5 +120,5 @@
       <update_rate>10</update_rate>
       <visualize>1</visualize>
-      <topic>rgb_image</topic>
+      <topic>${topic_prefix}rgb_image</topic>
     </sensor>
   </gazebo>
@@ -164,5 +170,5 @@
       <update_rate>10</update_rate>
       <visualize>1</visualize>
-      <topic>camera/realsense2_camera_node/depth/image_rect_gazebo_raw</topic>
+      <topic>${topic_prefix}camera/realsense2_camera_node/depth/image_rect_gazebo_raw</topic>
     </sensor>
     <sensor name="head_rgb_camera" type="camera">
@@ -184,5 +190,5 @@
       <update_rate>30</update_rate>
       <visualize>1</visualize>
-      <topic>camera/realsense2_camera_node/color/image_raw</topic>
+      <topic>${topic_prefix}camera/realsense2_camera_node/color/image_raw</topic>
     </sensor>
   </gazebo>

File: go2_gazebo_sim/go2_description/urdf/unitree_go2_robot.xacro (robot description, xacro)
@@ -3,4 +3,9 @@
     xmlns:xacro="http://www.ros.org/wiki/xacro">
     <xacro:arg name="DEBUG" default="false"/>
+    <!-- Robot namespace for multi-robot support (e.g., "robot1", "robot2") -->
+    <xacro:arg name="robot_namespace" default=""/>
+    <xacro:property name="ns" value="$(arg robot_namespace)"/>
+    <!-- Topic prefix: empty if no namespace, otherwise "namespace/" -->
+    <xacro:property name="topic_prefix" value="${ns + '/' if ns != '' else ''}"/>
     <xacro:include filename="$(find go2_description)/urdf/const.xacro"/>
     <xacro:include filename="$(find go2_description)/urdf/materials.xacro"/>

File: go2_gazebo_sim/go2_description/urdf/velodyne.xacro (robot description, xacro)
@@ -51,7 +51,7 @@
         <sensor name="velodyne-VLP16" type="gpu_lidar">
             <pose>0 0 0 0 0 0</pose>
-            <topic>scan</topic>
+            <topic>${topic_prefix}scan</topic>
             <update_rate>10</update_rate>
-            <gz_frame_id>laser</gz_frame_id>
+            <gz_frame_id>${topic_prefix}laser</gz_frame_id>
             <lidar>
                 <scan>
@@ -79,5 +79,5 @@
                     <stddev>0.008</stddev>
                 </noise>
-                <frame_id>laser</frame_id>
+                <frame_id>${topic_prefix}laser</frame_id>
             </lidar>
             <visualize>true</visualize>
