Commit message: Adjust camera angle

File: unitree/go2_gazebo_sim/go2_description/urdf/unitree_go2_robot.xacro (robot description, xacro)
@@ -107,5 +107,5 @@
         <parent link="trunk"/>
         <child link="camera_link"/>
-        <origin rpy="0 0.6109 0" xyz="0.33 0 0.085"/>
+        <origin rpy="0 0.436332 0" xyz="0.33 0 0.085"/>
     </joint>
     <!-- <joint name="lidar_l1_joint" type="fixed">
